File: asmTest.kicad_sch (KiCad schematic)
At the start: 3 parts, among them U1 LM5109ASD, U2 LM5109ASD, U3 LM5109ASD

Commit message: first iteration of test
Parts:
- added C1, C3, C5: 100n, Capacitor_SMD:C_0603_1608Metric, symbol Device:C
- added C10: 2u2, Capacitor_SMD:C_1206_3216Metric, symbol Device:C
- added C2, C4, C6: 1u, Capacitor_SMD:C_1206_3216Metric, symbol Device:C
- added C7: 100u/100V, Capacitor_THT:CP_Radial_D10.0mm_P5.00mm, symbol Device:C_Polarized
- added FID1, FID2: Fiducial, Fiducial:Fiducial_1mm_Mask3mm, symbol Mechanical:Fiducial
- added J1: Conn_01x08_Pin, Connector_PinSocket_2.54mm:PinSocket_1x08_P2.54mm_Vertical, symbol Connector:Conn_01x08_Pin
- added J4: Conn_01x02_Pin, Connector_PinHeader_2.54mm:PinHeader_1x02_P2.54mm_Vertical, symbol Connector:Conn_01x02_Pin
- added J5: Conn_01x03_Socket, Connector_PinSocket_2.54mm:PinSocket_1x03_P2.54mm_Horizontal, symbol Connector:Conn_01x03_Socket
- added LOGO1: var1, Symbol:OSHW-Logo2_9.8x8mm_Copper, symbol Graphic:Logo_Open_Hardware_Small
- added Q1, Q2, Q3, Q4, Q5, Q6: BSC026N08, Package_TO_SOT_SMD:TDSON-8-1, symbol Transistor_FET:BSC035N10NS5
- added R1, R2, R3, R4, R5, R6: 33R, Resistor_SMD:R_0603_1608Metric, symbol Device:R
- added R7, R8: 0.001R, Resistor_SMD:R_2512_6332Metric, symbol Device:R
- added U4: SN65HVD1050D, Package_SO:SOIC-8_3.9x4.9mm_P1.27mm, symbol Interface_CAN_LIN:SN65HVD1050D
- added U5: ADuM121N, Package_SO:SOIC-8_3.9x4.9mm_P1.27mm, symbol Isolator:ADuM121N
- added U6: ATmega328P-P, Package_DIP:DIP-28_W7.62mm, symbol MCU_Microchip_ATmega:ATmega328P-P
- U1, U2, U3: value LM5109ASD -> LM5109BSD; def Datasheet (none) -> http://www.ti.com/lit/ds/symlink/lm5109a.pdf; def Value (none) -> LM5109ASD; var1 Value (none) -> LM5109BSD
Connections:
- net +10V: now reaches U3.1 (VDD)
- net +10V: now also U1.1 (VDD), U2.1 (VDD), C2.1, C4.1, C6.1, J1.1 (Pin_1)
- net hi_C: now reaches U3.2 (HI)
- net hi_C: now also U6.27 (PC4)
- net li_C: now reaches U3.3 (LI)
- net li_C: now also U6.28 (PC5)
- net GND: now reaches U3.4 (VSS), U3.9 (VSS)
- net GND: now also U1.4 (VSS), U1.9 (VSS), U2.4 (VSS), U2.9 (VSS), C10.2, C2.2, C4.2, C6.2, C7.2, J1.8 (Pin_8), J4.2 (Pin_2), Q2.1 (S), Q2.2 (S), Q2.3 (S), Q4.1 (S), Q4.2 (S), Q4.3 (S), Q6.1 (S), Q6.2 (S), Q6.3 (S), U4.2 (GND), U5.4 (GND1), U5.5 (GND2), U6.22 (GND), U6.8 (GND)
- net at U3.5 (LO): now also R6.1
- net at U3.6 (HS): now also C5.2, Q5.1 (S), Q5.2 (S), Q5.3 (S), Q6.5 (D), R8.1
- net at U3.7 (HO): now also R5.1
- net at U3.8 (HB): now also C5.1
- net hi_A: now reaches U1.2 (HI)
- net hi_A: now also U6.23 (PC0)
- net li_A: now reaches U1.3 (LI)
- net li_A: now also U6.24 (PC1)
- net at U1.5 (LO): now also R2.1
- net at U1.6 (HS): now also C1.2, Q1.1 (S), Q1.2 (S), Q1.3 (S), Q2.5 (D), R7.1
- net at U1.7 (HO): now also R1.1
- net at U1.8 (HB): now also C1.1
- net hi_B: now reaches U2.2 (HI)
- net hi_B: now also U6.25 (PC2)
- net li_B: now reaches U2.3 (LI)
- net li_B: now also U6.26 (PC3)
- net at U2.5 (LO): now also R4.1
- net phase_B: now reaches U2.6 (HS)
- net phase_B: now also C3.2, J5.2 (Pin_2), Q3.1 (S), Q3.2 (S), Q3.3 (S), Q4.5 (D)
- net at U2.7 (HO): now also R3.1
- net at U2.8 (HB): now also C3.1
- new net: Q1.4 (G), R1.2
- new net: Q4.4 (G), R4.2
- new net: Q3.4 (G), R3.2
- new net: Q2.4 (G), R2.2
- new net: Q6.4 (G), R6.2
- new net: Q5.4 (G), R5.2
- new net +5V: C10.1, J1.2 (Pin_2), U4.3 (VCC), U5.1 (VDD1), U5.8 (VDD2), U6.20 (AVCC), U6.7 (VCC)
- new net +BATT: C7.1, J4.1 (Pin_1), Q1.5 (D), Q3.5 (D), Q5.5 (D)
- new net can_rx: U4.4 (RXD), U6.2 (PD0)
- new net can_tx: U4.1 (TXD), U6.3 (PD1)
- new net canh: J1.3 (Pin_3), U4.7 (CANH)
- new net canl: J1.4 (Pin_4), U4.6 (CANL)
- new net phase_A: J5.1 (Pin_1), R7.2
- new net phase_C: J5.3 (Pin_3), R8.2
- new net rx: J1.5 (Pin_5), U5.7 (VIA)
- new net tx: J1.6 (Pin_6), U5.6 (VOB)
- new net uart_rx: U5.2 (VOA), U6.4 (PD2)
- new net uart_tx: U5.3 (VIB), U6.5 (PD3)
- no-connect marks 0 -> 17
Other:
- moved on the sheet: U1

Commit message: add fictional LCSC PN to test switching of user-defined fields
Parts:
- C1, C3, C5: LCSC (none) -> C01; def LCSC (none) -> C01
- C10: LCSC (none) -> C04; def LCSC (none) -> C04
- C2, C4, C6: LCSC (none) -> C02; def LCSC (none) -> C02
- C7: LCSC (none) -> C03; def LCSC (none) -> C03
- J1: LCSC (none) -> C06; def LCSC (none) -> C06
- J4: LCSC (none) -> C07; def LCSC (none) -> C07
- J5: LCSC (none) -> C08; def LCSC (none) -> C08
- Q1, Q2, Q3, Q4, Q5, Q6: LCSC (none) -> C50; def LCSC (none) -> C10; var1 LCSC (none) -> C50; var2 LCSC (none) -> C70
- R1, R2, R3, R4, R5, R6: LCSC (none) -> C51; def LCSC (none) -> C11; var1 LCSC (none) -> C51; var2 LCSC (none) -> C71
- R7, R8: LCSC (none) -> C12; def LCSC (none) -> C12; var2 LCSC (none) -> C75
- U1, U2, U3: LCSC (none) -> C52; def LCSC (none) -> C13; var1 LCSC (none) -> C52
- U4: LCSC (none) -> C14; def LCSC (none) -> C14
- U5: LCSC (none) -> C15; def LCSC (none) -> C15
- U6: LCSC (none) -> C16; def LCSC (none) -> C16
